File: photodiode.kicad_sch (KiCad schematic)
At the start: 24 parts, among them J2 Conn_01x03, SW1 SW_Rotary_1x6_MP, U4 OPA210

Commit message: Save progress.
Parts:
- removed C20, C21, C22, C23, C24, C25: 10pF, Capacitor_SMD:C_0603_1608Metric_Pad1.08x0.95mm_HandSolder, symbol DK_Kemet_0603_Capacitors_X7R_E24:C_10pF_50V
- removed J2: Conn_01x03, Connector_PinHeader_1.27mm:PinHeader_1x02_P1.27mm_Vertical, symbol Connector_Generic:Conn_01x02
- removed R12: 0R, Resistor_SMD:R_0603_1608Metric_Pad0.98x0.95mm_HandSolder, symbol DK_Yageo_0603_Resistors_1%_100mW_ThinFilm:R_0R
- removed R15: 1K, Resistor_SMD:R_0603_1608Metric_Pad0.98x0.95mm_HandSolder, symbol DK_Yageo_0603_Resistors_1%_100mW_ThinFilm:R_1K
- removed R16: 3K, Resistor_SMD:R_0603_1608Metric_Pad0.98x0.95mm_HandSolder, symbol DK_Yageo_0603_Resistors_1%_100mW_ThinFilm:R_3K
- removed R17: 10K, Resistor_SMD:R_0603_1608Metric_Pad0.98x0.95mm_HandSolder, symbol DK_Yageo_0603_Resistors_1%_100mW_ThinFilm:R_10K
- removed R18: 30K, Resistor_SMD:R_0603_1608Metric_Pad0.98x0.95mm_HandSolder, symbol DK_Yageo_0603_Resistors_1%_100mW_ThinFilm:R_30K
- removed R19: 100K, Resistor_SMD:R_0603_1608Metric_Pad0.98x0.95mm_HandSolder, symbol DK_Yageo_0603_Resistors_1%_100mW_ThinFilm:R_100K
- removed R20: 150K, Resistor_SMD:R_0603_1608Metric_Pad0.98x0.95mm_HandSolder, symbol DK_Yageo_0603_Resistors_1%_100mW_ThinFilm:R_150K
- removed R21: 4K7, Resistor_SMD:R_0603_1608Metric_Pad0.98x0.95mm_HandSolder, symbol DK_Yageo_0603_Resistors_1%_100mW_ThinFilm:R_4K7
- removed R22: 51R, Resistor_SMD:R_0603_1608Metric_Pad0.98x0.95mm_HandSolder, symbol DK_Yageo_0603_Resistors_1%_100mW_ThinFilm:R_51R
- added C20, C21, C22, C23, C24, C25: 5.6pF, Capacitor_SMD:C_0402_1005Metric_Pad0.74x0.62mm_HandSolder, symbol DK_Murata_GRM_0402_Capacitors:C_5.6pF
- added J2: Conn_BNC, 1_Conn_RF:BNC_panel_mount, symbol 1_Conn_RF:BNC_panel_mount
- added R15: 1K, Resistor_SMD:R_0402_1005Metric_Pad0.72x0.64mm_HandSolder, symbol DK_Yageo_RC_0402_Resistors:R_1K
- added R16: 3K, Resistor_SMD:R_0402_1005Metric_Pad0.72x0.64mm_HandSolder, symbol DK_Yageo_RC_0402_Resistors:R_3K
- added R17: 10K, Resistor_SMD:R_0402_1005Metric_Pad0.72x0.64mm_HandSolder, symbol DK_Yageo_RC_0402_Resistors:R_10K
- added R19: 100K, Resistor_SMD:R_0402_1005Metric_Pad0.72x0.64mm_HandSolder, symbol DK_Yageo_RC_0402_Resistors:R_100K_4
- added R20: 150K, Resistor_SMD:R_0402_1005Metric_Pad0.72x0.64mm_HandSolder, symbol DK_Yageo_RC_0402_Resistors:R_150K
- added R21: 4K7, Resistor_SMD:R_0603_1608Metric_Pad0.98x0.95mm_HandSolder, symbol DK_Yageo_RC_0603_Resistors:R_4K7
- added R22: 51R, Resistor_SMD:R_0603_1608Metric_Pad0.98x0.95mm_HandSolder, symbol DK_Yageo_RC_0603_Resistors:R_51R
- added R5: 30K, Resistor_SMD:R_0402_1005Metric_Pad0.72x0.64mm_HandSolder, symbol DK_Yageo_RC_0402_Resistors:R_30K
- R13: symbol DK_Yageo_0603_Resistors_1%_100mW_ThinFilm:R_0R -> DK_Yageo_RC_0603_Resistors:R_0R0; DigiKey Part Number 311-0.0GRTR-ND -> 311-0.0HRTR-ND; Manufacturer Part Number RC0603JR-070RL -> RC0603FR-070RL
- R14: symbol DK_Yageo_0603_Resistors_1%_100mW_ThinFilm:R_0R -> DK_Yageo_RC_0603_Resistors:R_0R0; DigiKey Part Number 311-0.0GRTR-ND -> 311-0.0HRTR-ND; Manufacturer Part Number RC0603JR-070RL -> RC0603FR-070RL; now in the parts list
- SW1: now not fitted
Connections:
- net GND: now also J2.2 (Ext), R21.1
- net at U4.1: now also C20.2, C21.2, C22.2, C23.2, C24.2, C25.2, R15.1, R16.1, R17.1, R19.1, R20.1, R21.2, R22.1, R5.1
- net at SW1.6: now also C25.1, R20.2
- net at SW1.1: now also C24.1, R15.2
- net at C26.1: now also J2.1 (In), R22.2
- net at SW1.5: now also C20.1, R19.2
- net at SW1.3: now also C22.1, R17.2
- net at SW1.2: now also C23.1, R16.2
- net at SW1.4: now also C21.1, R5.2
Other:
- moved on the sheet: R13

Commit message: Added fabrication files. Board finalized.
Parts:
- C26: Package/Footprint (none) -> 0603
- D3: Type (none) -> thru-hole; now not fitted
