File: photodiode.kicad_sch (KiCad schematic)
At the start: 24 parts, among them J2 Conn_01x03, SW1 SW_Rotary_1x6_MP, U4 OPA210

Commit message: Update schematic and pcb. Add fab files.
Parts:
- removed J2: Conn_01x03, Connector_PinHeader_1.27mm:PinHeader_1x02_P1.27mm_Vertical, symbol Connector_Generic:Conn_01x02
- added J2: Conn_Coaxial, 1_Conn_RF:BNC_panel_mount, symbol 1_Conn_RF:BNC_panel_mount
- C20, C21, C22, C23, C24, C25, C26, R15, R16, R17, R18, R19, R20, R21, R22: Package/Footprint (none) -> 0603
- D3: now not fitted; now in the parts list
- SW1: now not fitted
Connections:
- net GND: now also J2.2 (Ext)
- net at C26.1, R22.2: now also J2.1 (In)
