File: photodiodes_kicadproject.kicad_pcb (KiCad board)
At the start: 4 copper layers, 55 x 30 mm, 61 parts, among them J1 Conn_01x03, J2 Conn_01x03, Q1 Si2319CDS, SW1 SW_Rotary_1x6_MP, U1 LM317_SOT-223, U2 LM337_SOT223, U3 TPS65131RGE, U4 OPA210

Commit message: Update schematic and pcb. Add fab files.
Parts:
- J2: value Conn_01x03 -> Conn_Coaxial; footprint Connector_PinHeader_1.27mm:PinHeader_1x02_P1.27mm_Vertical -> 1_Conn_RF:BNC_panel_mount
- moved J2 2.81 mm to (140.0, 93.5)
Routing:
- net GND: track 18.4 -> 21.4 mm, vias 13 -> 15
- net Net-(J2-In): track 9.31 -> 9.97 mm
Other:
- board text added: "+5V Power In"
